File: custom_minimal_kicad/custom_pico_minimal.kicad_pcb (KiCad board)
At the start: 2 copper layers, 50 x 32 mm, 34 parts, among them J1 USB4085, J2 SWD, SW1 BOOTSEL, SW2 RESET, U1 NCP1117-3.3_SOT223, U2 W25Q128JVS, U3 RP2040, U4 SRV05-4, X1 ABM8-272-T3

Commit message: Add files via upload
Parts:
- D1: footprint Pico_Footprint_Library:LED_3mm -> Pico_Footprint_Library:LED_0805_2012Metric
- J1: value USB4085 -> USB4930-00-A; footprint Pico_Footprint_Library:USB_C_Receptacle_GCT_USB4085_improved -> Pico_Footprint_Library:CONN_USB4930-00-A_GCT
- R10, R11: value 1k -> 5.1k
- R3, R4: footprint Pico_Footprint_Library:0603-footprint-improved-Res3D -> Pico_Footprint_Library:0402-footprint-improved-Res3D
- U4: footprint Pico_Footprint_Library:SOT23-6 -> Pico_Footprint_Library:SOT23-6-SRV05-04
- moved J1 8.11 mm to (68.8, 100.0)
- moved R10 7.72 mm to (79.5, 104.5), turned to 180 degrees
- moved R4 2.73 mm to (93.1, 98.5), turned to 0 degrees
- moved R3 0.60 mm to (93.1, 99.5)
- moved U4 0.50 mm to (80.2, 100.0)
- moved D1 0.40 mm to (102.7, 86.9)
- moved C8 0.22 mm to (93.6, 96.8)
Connections:
- U4 pad 1: /USB_D- -> /USB_D+
- U4 pad 6: /USB_D+ -> /USB_D-
Routing:
- net Net-(J1-CC2): track 10.7 -> 6.23 mm
- net Net-(U3-USB_DM): track 7.37 -> 3.08 mm
- net GND: track 44.3 -> 47.8 mm, vias 50 -> 55
- net /USB_D+: track 19.2 -> 21.6 mm
- net VBUS: track 10.5 -> 9.20 mm
- net /USB_D-: track 19.0 -> 19.8 mm
- net Net-(D1-A): track 3.08 -> 3.89 mm
- net +3V3: track 73.5 -> 72.7 mm
- net Net-(J1-CC1): track 7.97 -> 8.11 mm, vias 0 -> 2

Commit message: Add files via upload
Parts:
- moved J1 5.00 mm to (73.8, 100.0)
- turned U4 to 0 degrees
