File: custom_minimal_kicad/custom_pico_minimal.kicad_sch (KiCad schematic)
At the start: 34 parts, among them J1 USB4085, J2 SWD, SW1 BOOTSEL, SW2 RESET, U1 NCP1117-3.3_SOT223, U2 W25Q128JVS, U3 RP2040, U4 SRV05-4, X1 ABM8-272-T3

Commit message: Add files via upload
Parts:
- removed D1: LED, Pico_Footprint_Library:LED_3mm, symbol Pico_Symbol_Library:LED
- removed J1: USB4085, Pico_Footprint_Library:USB_C_Receptacle_GCT_USB4085_improved, symbol Pico_Symbol_Library:USB_C_Receptacle_USB4085-improved
- added D1: LED, Pico_Footprint_Library:LED_0805_2012Metric, symbol Pico_Symbol_Library:LED_0805
- added J1: USB4930-00-A, Pico_Footprint_Library:CONN_USB4930-00-A_GCT, symbol Pico_Symbol_Library:USB4930-00-A
- R10, R11: value 1k -> 5.1k; LCSC Part # C852624 -> C723526
- R3, R4: footprint Pico_Footprint_Library:0603-footprint-improved-Res3D -> Pico_Footprint_Library:0402-footprint-improved-Res3D
- U4: footprint Pico_Footprint_Library:SOT23-6 -> Pico_Footprint_Library:SOT23-6-SRV05-04
Connections:
- net GND: now also D1.1 (K), J1.A1B12 (GND), J1.B1A12 (GND), J1.S1 (SHIELD), J1.S2 (SHIELD), J1.S3 (SHIELD), J1.S4 (SHIELD)
- net USB_D+: now also U4.1 (IO1), J1.A6 (D+), J1.B6 (D+); no longer U4.6 (IO4)
- net USB_D-: now also U4.6 (IO4), J1.A7 (D-), J1.B7 (D-); no longer U4.1 (IO1)
- net VBUS: now also J1.A4B9 (VBUS), J1.B4A9 (VBUS)
- net at R8.1: now also D1.2 (A)
- net at R10.2: now also J1.A5 (CC1)
- net at R11.2: now also J1.B5 (CC2)

Commit message: Add files via upload
Parts:
- R3, R4: LCSC Part # C844545 -> C384351
Changed lines of the file:
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@@
 	)
 	(no_connect
-		(at 99.06 175.26)
+		(at 99.06 170.18)
 	)
 	(no_connect
@@
 			)
 		)
-		(property "LCSC Part #" "C844545"
+		(property "LCSC Part #" "C384351"
 			(at 160.02 162.56 90)
 			(hide yes)
@@
 			)
 		)
-		(property "LCSC Part #" "C844545"
+		(property "LCSC Part #" "C384351"
 			(at 160.02 160.02 90)
 			(hide yes)
